Commit message: Add files via upload

File: ros_tracked_robot/urdf/ros_tracked_robot.urdf (robot description, URDF)
Before this commit: robot ros_tracked_robot, 12 links, 11 joints
Links:
- link arm0: mass 0.398273847654276 -> 0.39827
- link arm1: mass 0.114672786058552 -> 0.11467
- link arm2: mass 0.0970492123410936 -> 0.097049
- link tracked_left: mass 0.0122203534541079 -> 0
- link tracked_right: mass 0.0122203534541079 -> 0.01222
- link wheel1: mass 0.0942477796076938 -> 0.094248
- link wheel2: mass 0.0942477796076938 -> 0.094248
- link wheel3: mass 0.0942477796076938 -> 0.094248
- link wheel4: mass 0.0942477796076938 -> 0.094248
Joints:
- joint arm0_joint: origin xyz=-0.113073481764877 0.0965559838073363 0.00452339044918062 rpy=1.5707963267949 0 0 -> xyz=-0.11307 0.096556 0.0045234 rpy=1.5708 0 0
- joint arm_2_joint: origin xyz=-0.0262642027796428 0.167958898699502 0.0500000000000025 rpy=0 0 0 -> xyz=-0.056769 0.16024 0.05 rpy=0 0 0
- joint camera_joint: origin xyz=-0.113073481764877 0.0165559838073364 0.0695233904491806 rpy=1.5707963267949 0 0 -> xyz=-0.11307 0.016556 0.069523 rpy=1.5708 0 3.1416
- joint imu_joint: origin xyz=-0.0130734817648772 0.0165559838073364 0.00452339044918062 rpy=1.5707963267949 0 0 -> xyz=-0.013073 0.016556 0.0045234 rpy=1.5708 0 3.1416
- joint tracked_left_joint: origin xyz=0 -0.0784440161926636 0 rpy=1.5707963267949 0 3.14159265358979 -> xyz=-0.031537 -0.078444 0.053023 rpy=1.5708 0 0
- joint tracked_right_joint: origin xyz=0 0.111555983807336 0 rpy=1.5707963267949 0 3.14159265358979 -> xyz=-0.031537 0.11156 0.053023 rpy=1.5708 0 0
- joint wheel1_joint: origin xyz=0.0369265182351228 0.126555983807336 0.0195233904491806 rpy=1.5707963267949 0 0 -> xyz=0.036927 0.12656 0.019523 rpy=1.5708 0 0
- joint wheel2_joint: origin xyz=-0.0630734817648772 0.126555983807336 0.0195233904491807 rpy=1.5707963267949 0 0 -> xyz=-0.063073 0.12656 0.019523 rpy=1.5708 0 0
- joint wheel3_joint: origin xyz=-0.0630734817648772 -0.0934440161926637 0.0195233904491806 rpy=1.5707963267949 0 0 -> xyz=-0.063073 -0.093444 0.019523 rpy=1.5708 0 0
- joint wheel4_joint: origin xyz=0.0369265182351228 -0.0934440161926637 0.0195233904491807 rpy=1.5707963267949 0 0 -> xyz=0.036927 -0.093444 0.019523 rpy=1.5708 0 0

Commit message: Add files via upload

File: ros_tracked_robot/urdf/ros_tracked_robot.urdf (robot description, URDF)
Before this commit: robot ros_tracked_robot, 12 links, 11 joints
Links:
- added link dummy_root_link
Joints:
- added joint dummy_joint: type fixed, parent dummy_root_link, child base_link, origin xyz=0 0 0 rpy=0 0 0
- joint arm_1_joint: limit lower=0 upper=0 effort=0 velocity=0 -> lower=-1.5707963267949 upper=1.5707963267949 effort=100 velocity=10
- joint arm_2_joint: limit lower=0 upper=0 effort=0 velocity=0 -> lower=-1.5707963267949 upper=1.5707963267949 effort=100 velocity=10

Commit message: Add files via upload

File: ros_tracked_robot/urdf/ros_tracked_robot.urdf (robot description, URDF)
Before this commit: robot ros_tracked_robot, 13 links, 12 joints
Links:
- link tracked_left: geometry visual mesh filename=package://ros_tracked_robot/meshes/tracked_left.STL
- link tracked_right: mass 0.01222 -> 0; geometry visual mesh filename=package://ros_tracked_robot/meshes/tracked_right.STL
